File: HackPad.kicad_sch (KiCad schematic)
At the start: 28 parts, among them J1 Conn_ARM_SWD_TagConnect_TC2030, SW9 RotaryEncoder_Switch, U1 XIAO-RP2040-DIP

Commit message: Sketch done, busy with PCB
Parts:
- removed J1: Conn_ARM_SWD_TagConnect_TC2030, Connector:Tag-Connect_TC2030-IDC-FP_2x03_P1.27mm_Vertical, symbol Connector:Conn_ARM_SWD_TagConnect_TC2030
- added U2: ~, OLED:SSD1306-0.91-OLED-4pin-128x32, symbol oled:oled0.91
- SW A1: footprint (none) -> Button_Switch_Keyboard:SW_Cherry_MX_1.00u_PCB
- SW A2: footprint (none) -> Button_Switch_Keyboard:SW_Cherry_MX_1.00u_PCB
- SW A3: footprint (none) -> Button_Switch_Keyboard:SW_Cherry_MX_1.00u_PCB
- SW A4: footprint (none) -> Button_Switch_Keyboard:SW_Cherry_MX_1.00u_PCB
- SW B1: footprint (none) -> Button_Switch_Keyboard:SW_Cherry_MX_1.00u_PCB
- SW B2: footprint (none) -> Button_Switch_Keyboard:SW_Cherry_MX_1.00u_PCB
- SW B3: footprint (none) -> Button_Switch_Keyboard:SW_Cherry_MX_1.00u_PCB
- SW B4: footprint (none) -> Button_Switch_Keyboard:SW_Cherry_MX_1.00u_PCB
- SW9: footprint (none) -> Rotary_Encoder:RotaryEncoder_Alps_EC12E-Switch_Vertical_H20mm
- U1: footprint Module:MOUDLE14P-XIAO-DIP-SMD -> OPL:XIAO-RP2040-DIP
Connections:
- net GND: now also U2.1 (GND)
- net SCL: now also U2.4 (SDA)
- net SDA: now also U2.3 (SCL)
- net + 5V renamed +5V
- net +5V: now also U2.2 (VCC)
- no-connect marks 0 -> 2
