File: HackPad.kicad_pcb (KiCad board)
At the start: 2 copper layers, 28 parts, among them SW9 RotaryEncoder_Switch, U1 XIAO-RP2040-DIP

Commit message: diodes
Parts:
- moved D13 68.4 mm to (104.5, 155.0), turned to -90 degrees
- moved D9 59.7 mm to (105.0, 129.2), turned to -90 degrees
- moved D16 53.4 mm to (182.5, 155.4), turned to -90 degrees
- moved D14 51.7 mm to (130.5, 154.9), turned to -90 degrees
- moved D15 45.4 mm to (156.7, 154.9), turned to -90 degrees
- moved D12 44.5 mm to (182.5, 128.9), turned to -90 degrees
- moved D10 41.2 mm to (130.5, 129.2), turned to -90 degrees
- moved D11 34.2 mm to (157.0, 129.2), turned to -90 degrees

Commit message: 12/12
Parts:
- added G***: LOGO, Images:Hack Club, B.Cu at (172.5, 74.5)
- D10, D11, D12, D13, D14, D15, D16, D17, D9: moved to B.Cu
- moved U2 59.7 mm to (125.1, 72.7)
- moved D5 48.4 mm to (171.1, 134.3)
- moved SW B4 48.3 mm to (173.7, 117.3)
- moved SW9 46.6 mm to (166.5, 76.0)
- moved D4 45.9 mm to (171.1, 110.9)
- moved SW A4 45.9 mm to (173.7, 93.9)
- moved SW B3 45.3 mm to (154.6, 117.3)
- moved D6 45.2 mm to (152.1, 134.3)
- moved D7 43.1 mm to (133.0, 134.3)
- moved SW B2 43.1 mm to (135.6, 117.3)
- moved SW A3 42.7 mm to (154.6, 93.9)
- moved D3 42.6 mm to (152.1, 110.9)
- moved D16 42.2 mm to (161.9, 118.6)
- moved SW B1 42.0 mm to (116.5, 117.3)
- moved D8 42.0 mm to (114.0, 134.3)
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Routing:
- net GND: track 0.00 -> 255.2 mm, vias 0 -> 2
- net +5V: track 0.00 -> 228.5 mm, vias 0 -> 9
- net SW B: track 0.00 -> 105.6 mm
- net SW 4: track 0.00 -> 96.6 mm, vias 0 -> 4
- net SW A: track 0.00 -> 81.7 mm
- net SW 1: track 0.00 -> 79.5 mm, vias 0 -> 2
- net SW 3: track 0.00 -> 63.7 mm, vias 0 -> 3
- net SCL: track 0.00 -> 57.4 mm, vias 0 -> 2
- net SDA: track 0.00 -> 57.0 mm, vias 0 -> 2
- net LEDs: track 0.00 -> 55.8 mm, vias 0 -> 1
- net DIAL A: track 0.00 -> 52.6 mm, vias 0 -> 1
- net DIAL B: track 0.00 -> 48.5 mm
- net SW 2: track 0.00 -> 44.8 mm, vias 0 -> 1
- net DIAL S1: track 0.00 -> 37.9 mm
- net Net-(D4-DOUT): track 0.00 -> 32.5 mm
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Other:
- board outline added: 86.5 x 73.5 mm
- board text added: "RIOSPAD"
- board text added: "SilverFantom"
- board text added: "XIAO HERE"
